File: pcb/JTAG_hat/JTAG_hat.kicad_sch (KiCad schematic)
At the start: 44 parts, among them IC1 TPS563240DDCR, J1 GPIO, J2 Conn_ARM_JTAG_SWD_20, J3 Conn_ARM_JTAG_SWD_10, J4 Barrel_Jack_Switch, Q1 BSS138, Q2 BSS138, U1 CAT24C256, U2 SN74LVC2T45DCUR, U3 SN74LVC2T45DCUR, U4 SN74LVC2T45DCUR, U5 SN74LVC2T45DCUR, U6 74LVC2G240, U7 BQ29209DRBR

Commit message: Added battery charging, balancing, and protection circuits; 3D models
Parts:
- added C11: 0.022u, symbol Device:C_Small
- added C12: 4.7u, symbol Device:C_Small
- added C13, C15, C19, C20: 0.1u, symbol Device:C_Small
- added C14, C17: 10u, symbol Device:C_Small
- added C16, C18: 1u, symbol Device:C_Small
- added IC2: LTC4162EUFD-LAD#PBF, JTAG_hat:QFN50P400X500X80-29N-D, symbol JTAG_hat:LTC4162EUFD-LAD#PBF
- added L1: SRP4020FA-2R0M, JTAG_hat:SRP4020FA2R0M, symbol Device:L_Small
- added Q3: ECH8693R-TL-W, JTAG_hat:SOTFL65P280X95-8N, symbol JTAG_hat:ECH8693R-TL-W
- added Q4: PMV16XNR, JTAG_hat:SOT95P230X110-3N, symbol JTAG_hat:PMV16XNR
- added Q5: BSS138, Package_TO_SOT_SMD:SOT-23, symbol Transistor_FET:BSS138
- added R15: MFL0805R0100FS, Resistor_SMD:R_0805_2012Metric_Pad1.20x1.40mm_HandSolder, symbol Device:R_Small
- added R16: LVM06FTR015E-TR, Resistor_SMD:R_0603_1608Metric_Pad0.98x0.95mm_HandSolder, symbol Device:R_Small
- added R17, R18, R20, R21, R27: 10k, Resistor_SMD:R_0603_1608Metric_Pad0.98x0.95mm_HandSolder, symbol Device:R_Small
- added R19: 47k, Resistor_SMD:R_0603_1608Metric_Pad0.98x0.95mm_HandSolder, symbol Device:R_Small
- added R22: 1k, Resistor_SMD:R_0603_1608Metric_Pad0.98x0.95mm_HandSolder, symbol Device:R_Small
- added R23, R24: 100E, Resistor_SMD:R_0603_1608Metric_Pad0.98x0.95mm_HandSolder, symbol Device:R_Small
- added R25: 260E, Resistor_SMD:R_0603_1608Metric_Pad0.98x0.95mm_HandSolder, symbol Device:R_Small
- added R26: 160E, Resistor_SMD:R_0603_1608Metric_Pad0.98x0.95mm_HandSolder, symbol Device:R_Small
- added TH1: NTCS0402E3103JL1T, symbol Device:Thermistor_NTC
- C1, C10, C2, C3, C4, C5, C6, C7, C8, C9: footprint Capacitor_SMD:C_0603_1608Metric_Pad1.08x0.95mm_HandSolder -> (none)
- D2: footprint (none) -> LED_SMD:LED_0603_1608Metric_Pad1.05x0.95mm_HandSolder
- F1: footprint (none) -> Resistor_SMD:R_0603_1608Metric_Pad0.98x0.95mm_HandSolder
Connections:
- net +12V: now also C15.1, IC2.7 (VIN), Q3.1 (S)
- net +3.3V: now also IC2.15 (DVCC), R19.2, R20.2, R21.2
- net GND: now also BT2.2 (-), U7.5 (GND), U7.9 (EPAD), C12.1, C13.1, C14.2, C15.2, C16.2, C17.2, C18.2, IC2.16 (SYNC), IC2.23 (PGND_1), IC2.24 (PGND_2), IC2.29 (AGND), Q5.2 (S), R18.1, TH1.2
- net GPIO2/SDA1: now also IC2.14 (SDA), R19.1
- net GPIO3/SCL1: now also IC2.13 (SCL), R20.1
- net GPIO4/GPCLK0: now also IC2.12 (~{SMBALERT}), R21.1
- net at BT1.1 (+): now also R26.2
- net at BT1.2 (-): now also BT2.1 (+), R24.1, R25.1
- net at U7.1 (VC2): now also C19.1, R26.1
- net at U7.2 (VC1): now also C19.2, C20.1, R25.2
- net at U7.3 (VC1_CB): now also C20.2, R24.2
- net at U7.4 (CD): now also C18.1
- net at U7.7 (VDD): now also R23.1
- net at U7.8 (OUT): now also R22.1
- new net: C13.2, IC2.3 (VOUTA)
- new net: Q4.2 (S), R23.2, R27.1
- new net: Q4.1 (G), Q5.3 (D), R27.2
- new net: C11.1, IC2.25 (SW_1), IC2.26 (SW_2), L1.1
- new net: IC2.21 (CSP), L1.2, Q3.3 (S), R16.2
- new net: C11.2, IC2.1 (BOOST)
- new net: IC2.6 (INFET), Q3.2 (G)
- new net: IC2.5 (CLP), Q3.7 (D), Q3.8 (D), R15.1
- new net: IC2.10 (NTC), R17.1, TH1.1
- new net: IC2.11 (RT), R18.2
- new net: IC2.22 (BATFET), Q3.4 (G)
- new net: IC2.9 (NTCBIAS), R17.2
- new net: Q5.1 (G), R22.2
- new net +BATT: C17.1, IC2.19 (BATSENS+), IC2.20 (CSN), Q4.3 (D), R16.1
- new net BC_INTVCC: C12.2, IC2.18 (CELLS1), IC2.2 (INTVCC)
- new net BC_VCC2P5: C16.1, IC2.17 (CELLS0), IC2.8 (VCC2P5)
- new net VS: C14.1, IC2.27 (VOUT_1), IC2.28 (VOUT_2), IC2.4 (CLN), Q3.5 (D), Q3.6 (D), R15.2
Other:
- note added: "Battery Charging, Balance, and Protection"
- note added: "ID_SD and ID_SC PINS: These pins are reserved for HAT ID EEPROM. DO NOT USE these pins for anything other than attaching an I2C ID EEPROM. Leave unconnected if ID EEPROM not required. At boot time this I2C interface will be interrogated to look for an EEPROM that identifes the attached board and allows automagic setup of the GPIOs (and optionally, Linux drivers). Bridging JP1 enables write protec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"
- note added: "JTAG Reset Output"
- note added: "Overvoltage Protection"
- note removed: "CHANGE LOCATION OF 3D FILES TO INSIDE PROJECT DIRECTORY"
- note removed: "ID_SD and ID_SC PINS: These pins are reserved for HAT ID EEPROM. At boot time this I2C interface will be interrogated to look for an EEPROM that identifes the attached board and allows automagic setup of the GPIOs (and optionally, Linux drivers). Bridging JP1 enables write protection. DO NOT USE these pins for anything other than attaching an I2C ID EEPROM. Leave unconnected if ID EEPROM not requ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"
- note removed: "Reset"
- moved on the sheet: BT1, BT2, C1, C10, C2, C3, C4, C5, C6, C7, C8, C9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
